File: telemetria-control/Controlador de Vuelo/PCB/AdaptadorD1/MainBoard_a/MainBoard_a.sch (KiCad schematic (older format))
At the start: 7 parts, among them J1 Conn_01x04, Q1 BC548, U1 WeMos_mini

Commit message: agrego tarea de testeo del buzzer
Parts:
- BT1: footprint (none) -> Componentes:Holder2032
- BZ1: footprint (none) -> Buzzers_Beepers:Buzzer_12x9.5RM7.6
- J1: footprint (none) -> Pin_Headers:Pin_Header_Angled_1x04_Pitch2.54mm
- R1, R2: footprint (none) -> Resistors_THT:R_Axial_DIN0207_L6.3mm_D2.5mm_P7.62mm_Horizontal
- U1: footprint (none) -> wemos_d1_mini:D1_mini_board
Changed lines of the file:
@@
 LIBS:valves
 LIBS:wemos_mini
+LIBS:MainBoard_a-cache
 EELAYER 25 0
 EELAYER END
@@
 F 0 "U1" H 5250 3250 60  0000 C CNN
 F 1 "WeMos_mini" H 5250 2250 60  0000 C CNN
-F 2 "" H 5800 2050 60  0000 C CNN
+F 2 "wemos_d1_mini:D1_mini_board" H 5800 2050 60  0001 C CNN
 F 3 "" H 5800 2050 60  0000 C CNN
 	1    5250 2750
@@
 F 0 "J1" H 1200 2600 50  0000 C CNN
 F 1 "Conn_01x04" H 1200 2100 50  0000 C CNN
-F 2 "" H 1200 2400 50  0001 C CNN
+F 2 "Pin_Headers:Pin_Header_Angled_1x04_Pitch2.54mm" H 1200 2400 50  0001 C CNN
 F 3 "" H 1200 2400 50  0001 C CNN
 	1    1200 2400
@@
 F 0 "R1" V 2580 4400 50  0000 C CNN
 F 1 "10k" V 2500 4400 50  0000 C CNN
-F 2 "" V 2430 4400 50  0001 C CNN
+F 2 "Resistors_THT:R_Axial_DIN0207_L6.3mm_D2.5mm_P7.62mm_Horizontal" V 2430 4400 50  0001 C CNN
 F 3 "" H 2500 4400 50  0001 C CNN
 	1    2500 4400
@@
 Buzzer
 $Comp
-L +3.3V #PWR2
+L +3.3V #PWR01
 U 1 1 5DAD0E24
 P 3100 3800
-F 0 "#PWR2" H 3100 3650 50  0001 C CNN
+F 0 "#PWR01" H 3100 3650 50  0001 C CNN
 F 1 "+3.3V" H 3100 3940 50  0000 C CNN
 F 2 "" H 3100 3800 50  0001 C CNN
@@
 $EndComp
 $Comp
-L GND #PWR3
+L GND #PWR02
 U 1 1 5DAD1024
 P 3100 4750
-F 0 "#PWR3" H 3100 4500 50  0001 C CNN
+F 0 "#PWR02" H 3100 4500 50  0001 C CNN
 F 1 "GND" H 3100 4600 50  0000 C CNN
 F 2 "" H 3100 4750 50  0001 C CNN
@@
 F 0 "BZ1" H 3400 4050 50  0000 L CNN
 F 1 "Buzzer" H 3400 3950 50  0000 L CNN
-F 2 "" V 3225 4100 50  0001 C CNN
+F 2 "Buzzers_Beepers:Buzzer_12x9.5RM7.6" V 3225 4100 50  0001 C CNN
 F 3 "" V 3225 4100 50  0001 C CNN
 	1    3250 4000
@@
 $EndComp
 $Comp
-L +3.3V #PWR6
+L +3.3V #PWR03
 U 1 1 5DAD2EBD
 P 5850 2300
-F 0 "#PWR6" H 5850 2150 50  0001 C CNN
+F 0 "#PWR03" H 5850 2150 50  0001 C CNN
 F 1 "+3.3V" H 5850 2440 50  0000 C CNN
 F 2 "" H 5850 2300 50  0001 C CNN
@@
 F 0 "R2" V 2880 4000 50  0000 C CNN
 F 1 "10k" V 2800 4000 50  0000 C CNN
-F 2 "" V 2730 4000 50  0001 C CNN
+F 2 "Resistors_THT:R_Axial_DIN0207_L6.3mm_D2.5mm_P7.62mm_Horizontal" V 2730 4000 50  0001 C CNN
 F 3 "" H 2800 4000 50  0001 C CNN
 	1    2800 4000
@@
 Connection ~ 3100 3850
 $Comp
-L GND #PWR1
+L GND #PWR04
 U 1 1 5DAD9B82
 P 1700 2700
-F 0 "#PWR1" H 1700 2450 50  0001 C CNN
+F 0 "#PWR04" H 1700 2450 50  0001 C CNN
 F 1 "GND" H 1700 2550 50  0000 C CNN
 F 2 "" H 1700 2700 50  0001 C CNN
@@
 F 0 "BT1" H 5050 4400 50  0000 L CNN
 F 1 "Battery_Cell" H 5050 4300 50  0000 L CNN
-F 2 "" V 4950 4360 50  0001 C CNN
+F 2 "Componentes:Holder2032" V 4950 4360 50  0001 C CNN
 F 3 "" V 4950 4360 50  0001 C CNN
 	1    4950 4300
@@
 $EndComp
 $Comp
-L GND #PWR5
+L GND #PWR05
 U 1 1 5DADBA2F
 P 4950 4500
-F 0 "#PWR5" H 4950 4250 50  0001 C CNN
+F 0 "#PWR05" H 4950 4250 50  0001 C CNN
 F 1 "GND" H 4950 4350 50  0000 C CNN
 F 2 "" H 4950 4500 50  0001 C CNN
@@
 $EndComp
 $Comp
-L +3.3V #PWR4
+L +3.3V #PWR06
 U 1 1 5DADBE5D
 P 4950 3950
-F 0 "#PWR4" H 4950 3800 50  0001 C CNN
+F 0 "#PWR06" H 4950 3800 50  0001 C CNN
 F 1 "+3.3V" H 4950 4090 50  0000 C CNN
 F 2 "" H 4950 3950 50  0001 C CNN
