File: telemetria-control/Controlador de Vuelo/PCB/AdaptadorD1/MainBoard_b/MainBoard_a.sch (KiCad schematic (older format))
At the start: 12 parts, among them J1 Conn_01x04, Q1 BC548, U1 WeMos_mini

Commit message: Esquematico version completa
Parts:
- gave numbers to parts that had none: 3
Changed lines of the file:
@@
 Buzzer
 $Comp
-L +3.3V #PWR01
+L +3.3V #PWR4
 U 1 1 5DAD0E24
 P 2200 4150
-F 0 "#PWR01" H 2200 4000 50  0001 C CNN
+F 0 "#PWR4" H 2200 4000 50  0001 C CNN
 F 1 "+3.3V" H 2200 4290 50  0000 C CNN
 F 2 "" H 2200 4150 50  0001 C CNN
@@
 $EndComp
 $Comp
-L GND #PWR02
+L GND #PWR5
 U 1 1 5DAD1024
 P 2200 5100
-F 0 "#PWR02" H 2200 4850 50  0001 C CNN
+F 0 "#PWR5" H 2200 4850 50  0001 C CNN
 F 1 "GND" H 2200 4950 50  0000 C CNN
 F 2 "" H 2200 5100 50  0001 C CNN
@@
 $EndComp
 $Comp
-L +3.3V #PWR03
+L +3.3V #PWR7
 U 1 1 5DAD2EBD
 P 8300 1850
-F 0 "#PWR03" H 8300 1700 50  0001 C CNN
+F 0 "#PWR7" H 8300 1700 50  0001 C CNN
 F 1 "+3.3V" H 8300 1990 50  0000 C CNN
 F 2 "" H 8300 1850 50  0001 C CNN
@@
 $EndComp
 $Comp
-L GND #PWR04
+L GND #PWR1
 U 1 1 5DAD9B82
 P 1700 2700
-F 0 "#PWR04" H 1700 2450 50  0001 C CNN
+F 0 "#PWR1" H 1700 2450 50  0001 C CNN
 F 1 "GND" H 1700 2550 50  0000 C CNN
 F 2 "" H 1700 2700 50  0001 C CNN
@@
 $EndComp
 $Comp
-L GND #PWR05
+L GND #PWR3
 U 1 1 5DADBA2F
 P 1700 6500
-F 0 "#PWR05" H 1700 6250 50  0001 C CNN
+F 0 "#PWR3" H 1700 6250 50  0001 C CNN
 F 1 "GND" H 1700 6350 50  0000 C CNN
 F 2 "" H 1700 6500 50  0001 C CNN
@@
 $EndComp
 $Comp
-L +3.3V #PWR06
+L +3.3V #PWR2
 U 1 1 5DADBE5D
 P 1700 5950
-F 0 "#PWR06" H 1700 5800 50  0001 C CNN
+F 0 "#PWR2" H 1700 5800 50  0001 C CNN
 F 1 "+3.3V" H 1700 6090 50  0000 C CNN
 F 2 "" H 1700 5950 50  0001 C CNN
@@
 $EndComp
 $Comp
-L Conn_01x05 J?
+L Conn_01x05 J2
 U 1 1 5DDDBA22
 P 9400 5350
-F 0 "J?" H 9400 5650 50  0000 C CNN
+F 0 "J2" H 9400 5650 50  0000 C CNN
 F 1 "Conn_01x05" H 9400 5050 50  0000 C CNN
 F 2 "" H 9400 5350 50  0001 C CNN
@@
 $EndComp
 $Comp
-L GND #PWR?
+L GND #PWR9
 U 1 1 5DDDF203
 P 9000 5650
-F 0 "#PWR?" H 9000 5400 50  0001 C CNN
+F 0 "#PWR9" H 9000 5400 50  0001 C CNN
 F 1 "GND" H 9000 5500 50  0000 C CNN
 F 2 "" H 9000 5650 50  0001 C CNN
@@
 $EndComp
 $Comp
-L +3V3 #PWR?
+L +3V3 #PWR8
 U 1 1 5DDDF7E7
 P 8950 5000
-F 0 "#PWR?" H 8950 4850 50  0001 C CNN
+F 0 "#PWR8" H 8950 4850 50  0001 C CNN
 F 1 "+3V3" H 8950 5140 50  0000 C CNN
 F 2 "" H 8950 5000 50  0001 C CNN
@@
 Acelerometro ADXL335\n
 $Comp
-L 4066 U?
+L 4066 U2
 U 1 1 5DDE2D81
 P 7950 4750
-F 0 "U?" H 8150 4601 50  0000 C CNN
+F 0 "U2" H 8150 4601 50  0000 C CNN
 F 1 "4066" H 8150 4900 50  0000 C CNN
 F 2 "" H 7950 4750 60  0001 C CNN
@@
 $EndComp
 $Comp
-L 4066 U?
+L 4066 U2
 U 2 1 5DDE349E
 P 7950 5400
-F 0 "U?" H 8150 5251 50  0000 C CNN
+F 0 "U2" H 8150 5251 50  0000 C CNN
 F 1 "4066" H 8150 5550 50  0000 C CNN
 F 2 "" H 7950 5400 60  0001 C CNN
@@
 $EndComp
 $Comp
-L 4066 U?
+L 4066 U2
 U 3 1 5DDE4223
 P 7950 6100
-F 0 "U?" H 8150 5951 50  0000 C CNN
+F 0 "U2" H 8150 5951 50  0000 C CNN
 F 1 "4066" H 8150 6250 50  0000 C CNN
 F 2 "" H 7950 6100 60  0001 C CNN
@@
 $EndComp
 $Comp
-L R R?
+L R R3
 U 1 1 5DDE9EDC
 P 7200 6100
-F 0 "R?" V 7280 6100 50  0000 C CNN
+F 0 "R3" V 7280 6100 50  0000 C CNN
 F 1 "10K" V 7200 6100 50  0000 C CNN
 F 2 "" V 7130 6100 50  0001 C CNN
@@
 $EndComp
 $Comp
-L GND #PWR?
+L GND #PWR6
 U 1 1 5DDEB1D8
 P 6950 6200
-F 0 "#PWR?" H 6950 5950 50  0001 C CNN
+F 0 "#PWR6" H 6950 5950 50  0001 C CNN
 F 1 "GND" H 6950 6050 50  0000 C CNN
 F 2 "" H 6950 6200 50  0001 C CNN
