File: telemetria-control/Controlador de Vuelo/PCB/AdaptadorD1/MainBoard_b/MainBoard_a.sch (KiCad schematic (older format))
At the start: 13 parts, among them J1 Conn_01x04, J2 Conn_01x05, J3 Conn_01x02, J4 Conn_01x08, J5 Conn_01x08, Q1 BC548, U1 WeMos_mini, U2 4066

Commit message: Error: se hizo una placa nueva arriba del proyecto de una vieja, Solucion:se restauro la version mas vieja y se creo la placa nueva en otra carpeta
Parts:
- removed J3: Conn_01x02, Connector_PinHeader_2.54mm:PinHeader_1x02_P2.54mm_Vertical, symbol Connector_Generic:Conn_01x02
- removed J4, J5: Conn_01x08, Connector_PinHeader_2.54mm:PinHeader_1x08_P2.54mm_Vertical, symbol Connector_Generic:Conn_01x08
- BT1: value CR2032-230mAh -> Battery_Cell; footprint (none) -> Componentes:Holder2032; symbol Device:Battery_Cell -> Battery_Cell
- BZ1: footprint Buzzer_Beeper:Buzzer_12x9.5RM7.6 -> Buzzers_Beepers:Buzzer_12x9.5RM7.6; symbol Device:Buzzer -> Buzzer
- J1: footprint Connector_PinHeader_2.54mm:PinHeader_1x04_P2.54mm_Vertical -> Pin_Headers:Pin_Header_Angled_1x04_Pitch2.54mm; symbol MainBoard_a-rescue:Conn_01x04 -> Conn_01x04
- J2: footprint Connector_PinHeader_2.54mm:PinHeader_1x05_P2.54mm_Vertical -> (none); symbol MainBoard_a-rescue:Conn_01x05 -> Conn_01x05
- Q1: footprint Package_TO_SOT_THT:TO-92L_Wide -> TO_SOT_Packages_THT:TO-92_Molded_Narrow; symbol MainBoard_a-rescue:BC548 -> BC548; Codigo TR1703130 -> (none); Encapsulado TO92 -> (none); Proveedor Elemon -> (none)
- R1, R2: footprint Resistor_SMD:R_1206_3216Metric -> Resistors_THT:R_Axial_DIN0207_L6.3mm_D2.5mm_P7.62mm_Horizontal; symbol Device:R -> R; Codigo RS3886245 -> (none); Encapsulado SMD 1206 -> (none); Proveedor Elemon -> (none)
- R3: footprint Resistor_SMD:R_1206_3216Metric -> (none); symbol Device:R -> R
- U1: footprint Module:WEMOS_D1_mini_light -> wemos_d1_mini:D1_mini_board; symbol MainBoard_a-rescue:WeMos_mini -> WeMos_mini
- U2: footprint Package_SO:SOIC-14_3.9x8.7mm_P1.27mm -> (none); symbol MainBoard_a-rescue:4066 -> 4066; Codigo CI2757372 -> (none); Encapsulado SOIC14.SMD -> (none); Proveedor Elemon -> (none)
- U2: footprint Package_SO:SOIC-14_3.9x8.7mm_P1.27mm -> (none); symbol MainBoard_a-rescue:4066 -> 4066; codigo proveedor CI2757372 -> (none); encapsulado SOIC14.SMD -> (none); proveedor Elemon -> (none)
Connections:
- net X_Sel: now also U2.13 (ON); no longer U1.11 (D0), U2.6 (ON)
- net Y_Sel: no longer U1.12 (D5)
- net Z_Sel: now also U2.6 (ON); no longer U1.13 (D6), U2.13 (ON)
- new net X_sel: U1.11 (D0)
- new net Y_sel: U1.12 (D5)
- new net Z_sel: U1.13 (D6)
Other:
- moved on the sheet: BT1, BZ1, J1, J2, Q1, R1, R2, R3, U1, U2A, U2B, U2C
