File: Control_Vuelo/Hardware/Adaptacion_D1_Mini/Kicad/MainBoard_a.kicad_pcb (KiCad board)
At the start: 2 copper layers, 45 x 45 mm, 14 parts, among them J1 Conn_01x04, J2 Conn_01x05, J3 Conn_01x02, J4 Conn_01x08, J5 Conn_01x08, Q1 BC548, U1 WeMos_mini, U2 4066

Commit message: Modificacion en la placa adaptacion_D1_mini en la pista de 3,3V
Parts:
- added ?: , kicad:UTN, F.Cu at (168.9, 115.6)
- added ?: , kicad:UTN, B.Cu at (170.8, 113.7)
- moved ? 24.4 mm to (163.8, 113.7)
- moved ? 0.64 mm to (174.0, 88.3)
Routing:
- net 3v3: track 112.2 -> 112.8 mm
Other:
- board text added: "24/4/2020 Rev2"
