File: Control_Vuelo/Hardware/Adaptacion_D1_Mini/Kicad/una_capa/MainBoard_a.kicad_pcb (KiCad board)
At the start: 2 copper layers, 45 x 45 mm, 27 parts, among them J1 Conn_01x04, J2 Desabilitar buzzer, J4 Conn_01x08, J5 Bateria, J6 Conn_01x08, J7 Llave, J8 Conn_01x05, Q1 BC817, U2 WeMos_mini, U3 4066

Commit message: Se corrigio un problema de superposicion en el PCB y se agregaron los Gerber
Parts:
- moved D1 3.18 mm to (57.8, 52.1), turned to 180 degrees
- turned R5 to 0 degrees
Routing:
- net Net-(D1-Pad2): track 1.91 -> 3.19 mm
- net 3v3: track 114.5 -> 115.5 mm
Changed lines of the file:
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@@
     (thickness 1.6)
     (drawings 4)
-    (tracks 152)
+    (tracks 156)
     (zones 0)
     (modules 27)
@@
     (visible_elements 7FFFFFFF)
     (pcbplotparams
-      (layerselection 0x00030_80000001)
+      (layerselection 0x018fc_ffffffff)
       (usegerberextensions false)
       (usegerberattributes false)
@@
       (outputformat 1)
       (mirror false)
-      (drillshape 1)
+      (drillshape 0)
       (scaleselection 1)
       (outputdirectory "./PCB_print"))
@@
   )
   (module LED_SMD:LED_0603_1608Metric (layer B.Cu)
-    (at 59.69 49.53 270)
+    (at 57.785 52.07 180)
     (descr "LED SMD 0603 (1608 Metric), square (rectangular) end terminal, IPC_7351 nominal, (Body size source: http://www.tortai-tech.com/upload/download/2011102023233369053.pdf), generated with kicad-footprint-generator")
     (tags diode)
     (attr smd)
-    (fp_text reference D1 (at 0 1.43 270) (layer B.SilkS)
-      (effects (font (size 1 1) (thickness 0.15)) (justify mirror))
-    )
-    (fp_text value LED (at 0 -1.43 270) (layer B.Fab)
+    (fp_text reference D1 (at 0 1.43 180) (layer B.SilkS)
+      (effects (font (size 1 1) (thickness 0.15)) (justify mirror))
+    )
+    (fp_text value LED (at 0 -1.43 180) (layer B.Fab)
       (effects (font (size 1 1) (thickness 0.15)) (justify mirror))
     )
@@
     (fp_line (start 1.48 0.73) (end 1.48 -0.73) (layer B.CrtYd) (width 0.05))
     (fp_line (start 1.48 -0.73) (end -1.48 -0.73) (layer B.CrtYd) (width 0.05))
-    (fp_text user %R (at 0 0 90) (layer B.Fab)
+    (fp_text user %R (at 0 0) (layer B.Fab)
       (effects (font (size 0.4 0.4) (thickness 0.06)) (justify mirror))
     )
-    (pad 1 smd roundrect (at -0.7875 0 270) (size 0.875 0.95) (layers B.Cu B.Paste B.Mask) (roundrect_rratio 0.25)
+    (pad 1 smd roundrect (at -0.7875 0 180) (size 0.875 0.95) (layers B.Cu B.Paste B.Mask) (roundrect_rratio 0.25)
       (net 3 "Net-(BZ1-Pad2)"))
-    (pad 2 smd roundrect (at 0.7875 0 270) (size 0.875 0.95) (layers B.Cu B.Paste B.Mask) (roundrect_rratio 0.25)
+    (pad 2 smd roundrect (at 0.7875 0 180) (size 0.875 0.95) (layers B.Cu B.Paste B.Mask) (roundrect_rratio 0.25)
       (net 13 "Net-(D1-Pad2)"))
     (model ${KISYS3DMOD}/LED_SMD.3dshapes/LED_0603_1608Metric.wrl
@@
   )
   (module Resistor_SMD:R_0603_1608Metric (layer B.Cu)
-    (at 57.785 49.53 270)
+    (at 57.785 49.53)
     (descr "Resistor SMD 0603 (1608 Metric), square (rectangular) end terminal, IPC_7351 nominal, (Body size source: http://www.tortai-tech.com/upload/download/2011102023233369053.pdf), generated with kicad-footprint-generator")
     (tags resistor)
     (attr smd)
-    (fp_text reference R5 (at 0 1.43 270) (layer B.SilkS)
-      (effects (font (size 1 1) (thickness 0.15)) (justify mirror))
-    )
-    (fp_text value 10k (at 0 -1.43 270) (layer B.Fab)
-      (effects (font (size 1 1) (thickness 0.15)) (justify mirror))
-    )
-    (fp_text user %R (at 0 0 270) (layer B.Fab)
+    (fp_text reference R5 (at 0 1.43) (layer B.SilkS)
+      (effects (font (size 1 1) (thickness 0.15)) (justify mirror))
+    )
+    (fp_text value 10k (at 0 -1.43) (layer B.Fab)
+      (effects (font (size 1 1) (thickness 0.15)) (justify mirror))
+    )
+    (fp_text user %R (at 0 0) (layer B.Fab)
       (effects (font (size 0.4 0.4) (thickness 0.06)) (justify mirror))
     )
@@
     (fp_line (start -0.8 0.4) (end 0.8 0.4) (layer B.Fab) (width 0.1))
     (fp_line (start -0.8 -0.4) (end -0.8 0.4) (layer B.Fab) (width 0.1))
-    (pad 2 smd roundrect (at 0.7875 0 270) (size 0.875 0.95) (layers B.Cu B.Paste B.Mask) (roundrect_rratio 0.25)
+    (pad 2 smd roundrect (at 0.7875 0) (size 0.875 0.95) (layers B.Cu B.Paste B.Mask) (roundrect_rratio 0.25)
       (net 13 "Net-(D1-Pad2)"))
-    (pad 1 smd roundrect (at -0.7875 0 270) (size 0.875 0.95) (layers B.Cu B.Paste B.Mask) (roundrect_rratio 0.25)
+    (pad 1 smd roundrect (at -0.7875 0) (size 0.875 0.95) (layers B.Cu B.Paste B.Mask) (roundrect_rratio 0.25)
       (net 1 3v3))
     (model ${KISYS3DMOD}/Resistor_SMD.3dshapes/R_0603_1608Metric.wrl
@@
   (segment (start 80.01 57.785) (end 80.645 58.42) (width 1) (layer B.Cu) (net 1) (status C00000))
   (segment (start 80.645 58.42) (end 85.09 58.42) (width 1) (layer B.Cu) (net 1) (status C00000))
-  (segment (start 57.785 48.7425) (end 57.3025 48.7425) (width 0.6) (layer B.Cu) (net 1) (status 400000))
-  (segment (start 49.53 59.055) (end 49.53 62.865) (width 0.6) (layer B.Cu) (net 1) (status 800000))
-  (segment (start 52.07 56.515) (end 49.53 59.055) (width 0.6) (layer B.Cu) (net 1))
-  (segment (start 53.34 56.515) (end 52.07 56.515) (width 0.6) (layer B.Cu) (net 1))
-  (segment (start 55.245 54.61) (end 53.34 56.515) (width 0.6) (layer B.Cu) (net 1))
-  (segment (start 55.245 50.8) (end 55.245 54.61) (width 0.6) (layer B.Cu) (net 1))
-  (segment (start 57.3025 48.7425) (end 55.245 50.8) (width 0.6) (layer B.Cu) (net 1))
-  (segment (start 57.785 48.7425) (end 57.9375 48.7425) (width 0.6) (layer B.Cu) (net 1) (status C00000))
-  (segment (start 57.9375 48.7425) (end 59.69 46.99) (width 0.6) (layer B.Cu) (net 1) (status 400000))
-  (segment (start 59.69 46.99) (end 65.405 46.99) (width 0.6) (layer B.Cu) (net 1))
-  (segment (start 65.405 46.99) (end 67.31 45.085) (width 0.6) (layer B.Cu) (net 1))
-  (segment (start 67.31 45.085) (end 72.39 45.085) (width 0.6) (layer B.Cu) (net 1))
-  (segment (start 72.39 45.085) (end 75.565 48.26) (width 0.6) (layer B.Cu) (net 1) (status 800000))
   (segment (start 49.53 62.865) (end 48.895 62.865) (width 0.6) (layer B.Cu) (net 1) (status C00000))
   (segment (start 56.515 83.82) (end 64.135 83.82) (width 0.6) (layer B.Cu) (net 1) (status 800000))
@@
   (segment (start 60.96 67.31) (end 60.96 77.47) (width 0.6) (layer B.Cu) (net 1))
   (segment (start 62.23 66.04) (end 60.96 67.31) (width 0.6) (layer B.Cu) (net 1))
+  (segment (start 49.53 62.865) (end 49.53 57.785) (width 0.6) (layer B.Cu) (net 1) (status 400000))
+  (segment (start 55.88 49.53) (end 56.9975 49.53) (width 0.6) (layer B.Cu) (net 1) (status 800000))
+  (segment (start 54.61 50.8) (end 55.88 49.53) (width 0.6) (layer B.Cu) (net 1))
+  (segment (start 54.61 52.705) (end 54.61 50.8) (width 0.6) (layer B.Cu) (net 1))
+  (segment (start 49.53 57.785) (end 54.61 52.705) (width 0.6) (layer B.Cu) (net 1))
+  (segment (start 56.9975 49.53) (end 56.9975 48.4125) (width 0.6) (layer B.Cu) (net 1) (status 400000))
+  (segment (start 75.565 46.99) (end 75.565 48.26) (width 0.6) (layer B.Cu) (net 1) (status 800000))
+  (segment (start 73.66 45.085) (end 75.565 46.99) (width 0.6) (layer B.Cu) (net 1))
+  (segment (start 65.405 45.085) (end 73.66 45.085) (width 0.6) (layer B.Cu) (net 1))
+  (segment (start 64.77 45.72) (end 65.405 45.085) (width 0.6) (layer B.Cu) (net 1))
+  (segment (start 62.865 47.625) (end 64.77 45.72) (width 0.6) (layer B.Cu) (net 1))
+  (segment (start 57.785 47.625) (end 62.865 47.625) (width 0.6) (layer B.Cu) (net 1))
+  (segment (start 56.9975 48.4125) (end 57.785 47.625) (width 0.6) (layer B.Cu) (net 1))
   (segment (start 53.34 60.96) (end 57.785 60.96) (width 1) (layer B.Cu) (net 2) (status C00000))
   (segment (start 49.53 65.405) (end 50.165 65.405) (width 1) (layer B.Cu) (net 2) (status C00000))
@@
   (segment (start 73.025 60.325) (end 73.025 61.595) (width 0.6) (layer B.Cu) (net 2))
   (segment (start 73.8125 59.5375) (end 73.025 60.325) (width 0.6) (layer B.Cu) (net 2))
-  (segment (start 59.69 48.7425) (end 62.7125 48.7425) (width 0.75) (layer B.Cu) (net 3) (status 400000))
-  (segment (start 62.7125 48.7425) (end 69.105 55.135) (width 0.75) (layer B.Cu) (net 3) (status 800000))
   (segment (start 73.93 54.61) (end 71.755 54.61) (width 0.75) (layer B.Cu) (net 3) (status 400000))
   (segment (start 71.23 55.135) (end 69.105 55.135) (width 0.75) (layer B.Cu) (net 3) (status 800000))
   (segment (start 71.755 54.61) (end 71.23 55.135) (width 0.75) (layer B.Cu) (net 3))
+  (segment (start 58.5725 52.07) (end 65.405 52.07) (width 0.6) (layer B.Cu) (net 3) (status 400000))
+  (segment (start 68.47 55.135) (end 69.105 55.135) (width 0.6) (layer B.Cu) (net 3) (status C00000))
+  (segment (start 65.405 52.07) (end 68.47 55.135) (width 0.6) (layer B.Cu) (net 3) (status 800000))
   (segment (start 53.34 71.12) (end 57.785 71.12) (width 1) (layer B.Cu) (net 4) (status C00000))
   (segment (start 49.53 67.945) (end 50.165 67.945) (width 1) (layer B.Cu) (net 4) (status C00000))
@@
   (segment (start 73.025 48.26) (end 69.63 48.26) (width 1) (layer B.Cu) (net 12) (status C00000))
   (segment (start 69.63 48.26) (end 69.105 47.735) (width 1) (layer B.Cu) (net 12) (status C00000))
-  (segment (start 57.785 50.3175) (end 59.69 50.3175) (width 0.6) (layer B.Cu) (net 13) (status C00000))
+  (segment (start 56.9975 52.07) (end 56.9975 51.5875) (width 0.6) (layer B.Cu) (net 13) (status 400000))
+  (segment (start 58.42 49.6825) (end 58.5725 49.53) (width 0.6) (layer B.Cu) (net 13) (status C00000))
+  (segment (start 58.42 50.165) (end 58.42 49.6825) (width 0.6) (layer B.Cu) (net 13) (status 800000))
+  (segment (start 56.9975 51.5875) (end 58.42 50.165) (width 0.6) (layer B.Cu) (net 13))
   (segment (start 53.34 76.2) (end 57.785 76.2) (width 1) (layer B.Cu) (net 14) (status C00000))
   (segment (start 53.34 73.66) (end 57.785 73.66) (width 1) (layer B.Cu) (net 15) (status C00000))
